Commit message: test

File: qube_bringup/urdf/controlled_qube.urdf.xacro (robot description, xacro)
@@ -1,5 +1,6 @@
 <?xml version="1.0"?>
-<robot name="qube" xmlns:xacro="http://www.ros.org/wiki/xacro">
+<robot name="qube_model" xmlns:xacro="http://www.ros.org/wiki/xacro">
     <xacro:include filename="$(find qube_description)/urdf/qube.macro.xacro"/>
+    <xacro:include filename="$(find qube_driver)/ros2_control/qube_driver.ros2_control.xacro"/>
     <link name="world"/>
     <xacro:qube prefix="qube_" base_x="0" base_y="0" base_z="0"/>
@@ -9,3 +10,4 @@
         <origin xyz="0 0 0" rpy="0 0 0"/>
     </joint>
+    <xacro:qube_driver_ros2_control name="qube_" prefix="qube_" baud_rate="115200" device="/dev/ttyACM0" simulation="false"/>
 </robot>

File: qube_description/urdf/qube.macro.xacro (robot description, xacro)
@@ -1,26 +1,21 @@
 <?xml version="1.0"?>
 <robot xmlns:xacro="http://www.ros.org/wiki/xacro">
-  <material name = "black">
-    <color rgba="0 0 0 1"/>
-  </material>
-  <material name = "red">
-    <color rgba="1 0 0 1"/>
-  </material>
-  <material name = "white">
-    <color rgba="1 1 1 1"/>
-  </material>
-	<xacro:macro name="qube_model" params="prefix base_x base_y base_z">
+	<xacro:macro name="qube" params="prefix base_x base_y base_z">
 		<xacro:property name="box_width" value="0.102"/>
 		<xacro:property name="angle_link_length" value="0.025"/>
 		<xacro:property name="angle_link_width" value="0.002"/>
-    <xacro:property name="angle_limit" value="3.14"/>
     <xacro:property name="rotor_radius" value="0.025"/>
     <xacro:property name="rotor_length" value="0.01"/>
-    <link name="${prefix}base_link"/>
-    <joint name="${prefix}base_joint" type="fixed">
-        <parent link="world"/>
-        <child link="${prefix}base_link"/>
-        <origin xyz="${base_x} ${base_y} ${base_z}" rpy="0 0 0"/>
-    </joint>
+    <material name = "black">
+      <color rgba="0 0 0 1"/>
+    </material>
+    <material name = "red">
+      <color rgba="1 0 0 1"/>
+    </material>
+    <material name = "white">
+      <color rgba="1 1 1 1"/>
+    </material>
+    <link name="${prefix}base_link">
+    </link>
 		<link name="${prefix}stator_link">
       <visual>
@@ -55,5 +50,5 @@
       <origin xyz="0 0 ${box_width/2}" rpy="0 0 0"/>
     </joint>
-    <joint name="${prefix}angle_joint" type="revolute">
+    <joint name="${prefix}motor_joint" type="revolute">
       <parent link="${prefix}stator_link"/>
       <child link="${prefix}rotor_link"/>

Commit message: needs tuning, possible bug with qube_controller_node

File: qube_bringup/urdf/controlled_qube.urdf.xacro (robot description, xacro)
@@ -4,10 +4,10 @@
     <xacro:include filename="$(find qube_driver)/ros2_control/qube_driver.ros2_control.xacro"/>
     <link name="world"/>
-    <xacro:qube prefix="qube_" base_x="0" base_y="0" base_z="0"/>
+    <xacro:qube prefix="" base_x="0" base_y="0" base_z="0"/>
     <joint name="world_to_base" type="fixed">
         <parent link="world"/>
-        <child link="qube_base_link"/>
+        <child link="base_link"/>
         <origin xyz="0 0 0" rpy="0 0 0"/>
     </joint>
-    <xacro:qube_driver_ros2_control name="qube_" prefix="qube_" baud_rate="115200" device="/dev/ttyACM0" simulation="false"/>
+    <xacro:qube_driver_ros2_control name="qube_" prefix="" baud_rate="115200" device="/dev/ttyACM0" simulation="false"/>
 </robot>

File: qube_description/urdf/qube.macro.xacro (robot description, xacro)
@@ -7,4 +7,5 @@
     <xacro:property name="rotor_radius" value="0.025"/>
     <xacro:property name="rotor_length" value="0.01"/>
+    <xacro:property name="leg_diameter" value="0.0102"/>
     <material name = "black">
       <color rgba="0 0 0 1"/>
@@ -15,4 +16,7 @@
     <material name = "white">
       <color rgba="1 1 1 1"/>
+    </material>
+    <material name = "blue">
+      <color rgba="0 0 1 1"/>
     </material>
     <link name="${prefix}base_link">
@@ -25,4 +29,22 @@
         <origin xyz="0 0 0" rpy="0 0 0"/>
         <material name="black"/>
+      </visual>
+    </link>
+   <link name ="${prefix}blue_lights_link">
+      <visual>
+        <geometry>
+          <box size="${box_width*1.01} ${box_width*1.01} ${box_width*0.1}"/>
+        </geometry>
+        <origin xyz="0 0 0" rpy="0 0 0"/>
+        <material name="blue"/>
+      </visual>
+    </link>
+    <link name="${prefix}red_stripe_link">
+      <visual>
+        <geometry>
+          <box size="${box_width*1.01} ${box_width*1.01} ${box_width*0.1}"/>
+        </geometry>
+        <origin xyz="0 0 0" rpy="0 0 0"/>
+        <material name="red"/>
       </visual>
     </link>
@@ -45,4 +67,14 @@
       </visual>
     </link>
+    <joint name="${prefix}blue_lights_joint" type="fixed">
+      <parent link="${prefix}stator_link"/>
+        <child link="${prefix}blue_lights_link"/>
+      <origin xyz="0 0 ${box_width*0.4}" rpy="0 0 0"/>
+    </joint>
+    <joint name="${prefix}red_stripe_joint" type="fixed">
+      <parent link="${prefix}stator_link"/>
+        <child link="${prefix}red_stripe_link"/>
+      <origin xyz="0 0 ${-box_width*0.4}" rpy="0 0 0"/>
+    </joint>
     <joint name="${prefix}stator_joint" type="fixed">
       <parent link="${prefix}base_link"/>
@@ -54,5 +86,5 @@
       <child link="${prefix}rotor_link"/>
       <origin xyz="0 0 ${box_width/2}" rpy="0 0 0"/>
-      <axis xyz="0 0 1"/>
+      <axis xyz="0 0 -1"/>
       <limit lower="-3.14" upper="3.14" effort="100.0" velocity="1.0"/>
     </joint>
